File: MCU Datalogger.kicad_pcb (KiCad board)
At the start: 2 copper layers, 50.2 x 35.6 mm, 30 parts, among them J1 Conn_01x04_Pin, J2 Conn_01x04_Pin, J3 Conn_01x09_Pin, J4 Conn_02x03_Odd_Even, U1 24LC1025, U2 24LC1025, U3 DS1337S_, U4 ATMEGA328P-AU, Y1 16 MHz, Y2 32.768 KHz

Commit message: Random changes for experimentation.
Parts:
- added G***: LOGO, Jacks Library 2:PCBImage, B.Cu at (95.3, 104.2)
